Commit message: clean up

File: cram_robots/cram_pr2_shopping_demo/resource/shelf.urdf (robot description, URDF)
Before this commit: robot shelve, 16 links, 15 joints
Links:
- removed link shelve_origin
- added link shelf_origin
Joints:
- removed joint left_leg_to_shelve_origin
- added joint left_leg_to_shelf_origin: type fixed, parent shelf_origin, child left_leg, origin xyz=0 -1.5 0
- joint origin_to_left_front_leg: parent shelve_origin -> shelf_origin
