Commit message: world-state-detecting with name

File: cram_robots/cram_pr2_shopping_demo/resource/kitchen.urdf (robot description, URDF)
Before this commit: robot iai_oven_area, 78 links, 77 joints
Links:
- removed link drawer_oven_right_back_link
- removed link drawer_oven_right_bottom_link
- removed link drawer_oven_right_top_link
- added link drawer_oven_right_board0_barrier_left_link, mass 1.0; collision box size=0.49 0.02 0.05; visual box size=0.49 0.02 0.05
- added link drawer_oven_right_board0_barrier_right_link, mass 1.0; collision box size=0.49 0.02 0.05; visual box size=0.49 0.02 0.05
- added link drawer_oven_right_board0_link, mass 1.0; collision box size=0.49 0.27 0.025; visual box size=0.49 0.27 0.025
- added link drawer_oven_right_board1_barrier_left_link, mass 1.0; collision box size=0.49 0.02 0.05; visual box size=0.49 0.02 0.05
- added link drawer_oven_right_board1_barrier_right_link, mass 1.0; collision box size=0.49 0.02 0.05; visual box size=0.49 0.02 0.05
- added link drawer_oven_right_board2_barrier_left_link, mass 1.0; collision box size=0.49 0.02 0.05; visual box size=0.49 0.02 0.05
- added link drawer_oven_right_board2_barrier_right_link, mass 1.0; collision box size=0.49 0.02 0.05; visual box size=0.49 0.02 0.05
- added link drawer_oven_right_board3_barrier_left_link, mass 1.0; collision box size=0.49 0.02 0.05; visual box size=0.49 0.02 0.05
- added link drawer_oven_right_board3_barrier_right_link, mass 1.0; collision box size=0.49 0.02 0.05; visual box size=0.49 0.02 0.05
- link drawer_oven_right_board1_link: geometry collision box size=0.49 0.27 0.025; visual box size=0.49 0.27 0.025
- link drawer_oven_right_board2_link: geometry collision box size=0.49 0.27 0.025; visual box size=0.49 0.27 0.025
- link drawer_oven_right_board3_link: geometry collision box size=0.49 0.27 0.025; visual box size=0.49 0.27 0.025
Joints:
- removed joint drawer_oven_right_back_joint
- removed joint drawer_oven_right_bottom_joint
- removed joint drawer_oven_right_top_joint
- added joint drawer_oven_right_board0_barrier_left_joint: type fixed, parent oven_area_area_right_drawer_main, child drawer_oven_right_board0_barrier_left_link, origin xyz=0 0.135 -0.62
- added joint drawer_oven_right_board0_barrier_right_joint: type fixed, parent oven_area_area_right_drawer_main, child drawer_oven_right_board0_barrier_right_link, origin xyz=0 -0.135 -0.62
- added joint drawer_oven_right_board0_joint: type fixed, parent oven_area_area_right_drawer_main, child drawer_oven_right_board0_link, origin xyz=0 0 -0.655
- added joint drawer_oven_right_board1_barrier_left_joint: type fixed, parent oven_area_area_right_drawer_main, child drawer_oven_right_board1_barrier_left_link, origin xyz=0 0.135 -0.295
- added joint drawer_oven_right_board1_barrier_right_joint: type fixed, parent oven_area_area_right_drawer_main, child drawer_oven_right_board1_barrier_right_link, origin xyz=0 -0.135 -0.295
- added joint drawer_oven_right_board2_barrier_left_joint: type fixed, parent oven_area_area_right_drawer_main, child drawer_oven_right_board2_barrier_left_link, origin xyz=0 0.135 0.035
- added joint drawer_oven_right_board2_barrier_right_joint: type fixed, parent oven_area_area_right_drawer_main, child drawer_oven_right_board2_barrier_right_link, origin xyz=0 -0.135 0.035
- added joint drawer_oven_right_board3_barrier_left_joint: type fixed, parent oven_area_area_right_drawer_main, child drawer_oven_right_board3_barrier_left_link, origin xyz=0 0.135 0.365
- added joint drawer_oven_right_board3_barrier_right_joint: type fixed, parent oven_area_area_right_drawer_main, child drawer_oven_right_board3_barrier_right_link, origin xyz=0 -0.135 0.365
- joint drawer_oven_right_board1_joint: origin xyz=0 0 -0.35 -> xyz=0 0 -0.33
- joint drawer_oven_right_board3_joint: origin xyz=0 0 0.35 -> xyz=0 0 0.33
- joint drawer_oven_right_front_joint: origin xyz=0.3 0 0 rpy=0 0. 0 -> xyz=0.25 0 0 rpy=0 0. 0
- joint oven_area_area_right_drawer_joint: axis (none) -> 0.999 0 0.044; limit (none) -> lower=0 upper=0.48 effort=300 velocity=10; origin xyz=0.7 0.45 0.05 rpy=0 0 0 -> xyz=0.02 0.44 0.05 rpy=0 0 0; type fixed -> prismatic
